File: Version1.brd (EAGLE design)
At the start: 51.5 x 35.5 mm, 42 parts, among them U1 MEGA328

Commit message: Minor updates to make the schematic cleaner
Connections:
- net GND: now also U$6.10, U$6.11, U$6.12, U$6.13, U$6.6, U$6.9; no longer U$6.GND@10, U$6.GND@11, U$6.GND@12, U$6.GND@13, U$6.GND@9, U$6.VSS@6
- net SD_CLK: now also U$6.5; no longer U$6.SCLK@5
- net SD_CS: now also U$6.2; no longer U$6.CS@2
- net SD_DI: now also U$6.3; no longer U$6.DI@3
- net SD_DO: now also U$6.7; no longer U$6.DO@7
- net VCC_AUX: now also U$6.4; no longer U$6.VDD@4
Changed lines of the file:
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@@
 <contactref element="U1" pad="3"/>
 <contactref element="U1" pad="5"/>
-<contactref element="U$6" pad="VSS@6"/>
-<contactref element="U$6" pad="GND@13"/>
-<contactref element="U$6" pad="GND@10"/>
-<contactref element="U$6" pad="GND@11"/>
-<contactref element="U$6" pad="GND@12"/>
-<contactref element="U$6" pad="GND@9"/>
+<contactref element="U$6" pad="6"/>
+<contactref element="U$6" pad="13"/>
+<contactref element="U$6" pad="10"/>
+<contactref element="U$6" pad="11"/>
+<contactref element="U$6" pad="12"/>
+<contactref element="U$6" pad="9"/>
 <via x="43.1" y="29.3" extent="1-16" drill="0.6" shape="square"/>
 <wire x1="43.37" y1="29.12" x2="43.19" y2="29.3" width="0.4064" layer="1"/>
@@
 <signal name="SD_DO">
 <contactref element="U1" pad="16"/>
-<contactref element="U$6" pad="DO@7"/>
+<contactref element="U$6" pad="7"/>
 <contactref element="U$7" pad="1"/>
 <via x="4.9" y="16" extent="1-16" drill="0.6" shape="square"/>
@@
 <signal name="SD_DI">
 <contactref element="U1" pad="15"/>
-<contactref element="U$6" pad="DI@3"/>
+<contactref element="U$6" pad="3"/>
 <contactref element="U$7" pad="4"/>
 <via x="5.4" y="20.5" extent="1-16" drill="0.6" shape="square"/>
@@
 <signal name="SD_CLK">
 <contactref element="U1" pad="17"/>
-<contactref element="U$6" pad="SCLK@5"/>
+<contactref element="U$6" pad="5"/>
 <contactref element="U$7" pad="3"/>
 <wire x1="3.2" y1="18.1" x2="3.1" y2="17.9" width="0.4064" layer="16"/>
@@
 <signal name="SD_CS">
 <contactref element="U1" pad="14"/>
-<contactref element="U$6" pad="CS@2"/>
+<contactref element="U$6" pad="2"/>
 <via x="6.4" y="21.7" extent="1-16" drill="0.6" shape="square"/>
 <wire x1="6.4" y1="21.7" x2="8.3" y2="19.8" width="0.4064" layer="1"/>
@@
 <contactref element="U$4" pad="3"/>
 <contactref element="U$2" pad="4"/>
-<contactref element="U$6" pad="VDD@4"/>
+<contactref element="U$6" pad="4"/>
 <contactref element="C4" pad="1"/>
 <contactref element="C10" pad="1"/>
